File: eagle/tco/analogTCO-RJ-alone-ext.sch (EAGLE design)
At the start: 20 parts, among them IC10 4515N, IC7 7805TV, IC9 4014N, J1 RJ11-2L-B

Commit message: Spravna verze schematu
Parts:
- removed J1: RJ11-2L-B, con-tycoelectronics:RJ11-2L-B
- added JP2: (no value), pinhead:PINHD-1X5
- added SJ1: (no value), jumper:SJ
- added XBUS: MAX487-P, rs232-rs485:MAX487-P
- SBUS: value MAX487-P -> RJ11-2L-B; device rs232-rs485:MAX487-P -> con-tycoelectronics:RJ11-2L-B
Connections:
- new net N$9: IC9A.SI, JP2.1, SJ1.1
- net GND: now also JP2.2, SBUS.2, SJ1.2, XBUSG$2.GND; no longer IC9A.SI, J1.2, SBUSG$2.GND
- net N$1: now also XBUSG$1.DE, XBUSG$1.RE/; no longer SBUSG$1.DE, SBUSG$1.RE/
- net N$2: now also XBUSG$1.RO; no longer SBUSG$1.RO
- net N$3: now also XBUSG$1.DI; no longer SBUSG$1.DI
- net N$4: now also SBUS.4, XBUSG$1.A; no longer J1.4, SBUSG$1.A
- net N$5: now also SBUS.3, XBUSG$1.B; no longer J1.3, SBUSG$1.B
- net N$70: now also JP2.4
- net N$71: now also JP2.5
- net N$8: now also SBUS.5; no longer J1.5
- net VCC: now also JP2.3, XBUSG$2.VCC; no longer SBUSG$2.VCC
Changed lines of the file:
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@@
 <parts>
 <part name="U$1" library="Arduino-clone" deviceset="NANO" device=""/>
-<part name="SBUS" library="rs232-rs485" deviceset="MAX487" device="-P"/>
+<part name="XBUS" library="rs232-rs485" deviceset="MAX487" device="-P"/>
 <part name="IC10" library="45xx" deviceset="4515" device="N"/>
 <part name="POWER" library="con-ptr500" deviceset="AK500/2" device=""/>
@@
 <part name="JP5" library="pinhead" deviceset="PINHD-1X2" device=""/>
 <part name="P+7" library="supply1" deviceset="VCC" device=""/>
-<part name="J1" library="con-tycoelectronics" deviceset="RJ11" device="" technology="-2L-B"/>
+<part name="SBUS" library="con-tycoelectronics" deviceset="RJ11" device="" technology="-2L-B"/>
 <part name="JP1" library="jumper" deviceset="JP1E" device=""/>
+<part name="JP2" library="pinhead" deviceset="PINHD-1X5" device=""/>
+<part name="P+6" library="supply1" deviceset="VCC" device=""/>
+<part name="SJ1" library="jumper" deviceset="SJ" device=""/>
 </parts>
 <sheets>
@@
 <instances>
 <instance part="U$1" gate="G$1" x="-111.76" y="10.16"/>
-<instance part="SBUS" gate="G$1" x="-7.62" y="-27.94"/>
+<instance part="XBUS" gate="G$1" x="-7.62" y="-27.94"/>
 <instance part="IC10" gate="A" x="-121.92" y="83.82" rot="MR0"/>
 <instance part="POWER" gate="-1" x="-210.82" y="-45.72"/>
@@
 <instance part="D2" gate="G$1" x="-185.42" y="-45.72"/>
 <instance part="P+5" gate="VCC" x="-116.84" y="-66.04"/>
-<instance part="GND5" gate="1" x="-218.44" y="86.36"/>
+<instance part="GND5" gate="1" x="-218.44" y="71.12"/>
 <instance part="IC9" gate="P" x="-254" y="-40.64"/>
 <instance part="IC10" gate="P" x="-246.38" y="-40.64"/>
-<instance part="SBUS" gate="G$2" x="-238.76" y="-40.64"/>
+<instance part="XBUS" gate="G$2" x="-238.76" y="-40.64"/>
 <instance part="GND6" gate="1" x="-106.68" y="81.28"/>
 <instance part="P+2" gate="VCC" x="17.78" y="-2.54"/>
@@
 <instance part="JP5" gate="G$1" x="-170.18" y="0" rot="R180"/>
 <instance part="P+7" gate="VCC" x="-160.02" y="12.7"/>
-<instance part="J1" gate="G$1" x="22.86" y="-63.5" rot="R270"/>
+<instance part="SBUS" gate="G$1" x="22.86" y="-63.5" rot="R270"/>
 <instance part="JP1" gate="A" x="5.08" y="-63.5" rot="R180"/>
+<instance part="JP2" gate="A" x="-195.58" y="91.44"/>
+<instance part="P+6" gate="VCC" x="-185.42" y="96.52"/>
+<instance part="SJ1" gate="1" x="-228.6" y="93.98"/>
 </instances>
 <busses>
@@
 <net name="N$1" class="0">
 <segment>
-<pinref part="SBUS" gate="G$1" pin="RE/"/>
+<pinref part="XBUS" gate="G$1" pin="RE/"/>
 <wire x1="-20.32" y1="-25.4" x2="-25.4" y2="-25.4" width="0.1524" layer="91"/>
 <wire x1="-25.4" y1="-25.4" x2="-25.4" y2="-30.48" width="0.1524" layer="91"/>
-<pinref part="SBUS" gate="G$1" pin="DE"/>
+<pinref part="XBUS" gate="G$1" pin="DE"/>
 <wire x1="-25.4" y1="-30.48" x2="-20.32" y2="-30.48" width="0.1524" layer="91"/>
 <wire x1="-25.4" y1="-30.48" x2="-68.58" y2="-30.48" width="0.1524" layer="91"/>
@@
 <net name="N$3" class="0">
 <segment>
-<pinref part="SBUS" gate="G$1" pin="DI"/>
+<pinref part="XBUS" gate="G$1" pin="DI"/>
 <wire x1="-20.32" y1="-35.56" x2="-71.12" y2="-35.56" width="0.1524" layer="91"/>
 <wire x1="-71.12" y1="-35.56" x2="-71.12" y2="5.08" width="0.1524" layer="91"/>
@@
 <wire x1="-246.38" y1="-50.8" x2="-238.76" y2="-50.8" width="0.1524" layer="91"/>
 <wire x1="-238.76" y1="-50.8" x2="-233.68" y2="-50.8" width="0.1524" layer="91"/>
-<pinref part="SBUS" gate="G$2" pin="GND"/>
+<pinref part="XBUS" gate="G$2" pin="GND"/>
 <wire x1="-238.76" y1="-48.26" x2="-238.76" y2="-50.8" width="0.1524" layer="91"/>
 <wire x1="-233.68" y1="-50.8" x2="-233.68" y2="-55.88" width="0.1524" layer="91"/>
@@
 </segment>
 <segment>
-<pinref part="IC9" gate="A" pin="SI"/>
-<wire x1="-248.92" y1="86.36" x2="-254" y2="86.36" width="0.1524" layer="91"/>
-<wire x1="-254" y1="86.36" x2="-254" y2="96.52" width="0.1524" layer="91"/>
-<wire x1="-254" y1="96.52" x2="-218.44" y2="96.52" width="0.1524" layer="91"/>
-<wire x1="-218.44" y1="96.52" x2="-218.44" y2="88.9" width="0.1524" layer="91"/>
-<pinref part="GND5" gate="1" pin="GND"/>
-</segment>
-<segment>
 <pinref part="IC10" gate="A" pin="INH"/>
 <pinref part="GND6" gate="1" pin="GND"/>
@@
 <wire x1="25.4" y1="-40.64" x2="38.1" y2="-40.64" width="0.1524" layer="91"/>
 <junction x="38.1" y="-40.64"/>
-<pinref part="J1" gate="G$1" pin="2"/>
+<pinref part="SBUS" gate="G$1" pin="2"/>
 <wire x1="25.4" y1="-40.64" x2="25.4" y2="-60.96" width="0.1524" layer="91"/>
+</segment>
+<segment>
+<pinref part="GND5" gate="1" pin="GND"/>
+<pinref part="JP2" gate="A" pin="2"/>
+<wire x1="-218.44" y1="93.98" x2="-218.44" y2="73.66" width="0.1524" layer="91"/>
+<wire x1="-198.12" y1="93.98" x2="-218.44" y2="93.98" width="0.1524" layer="91"/>
+<junction x="-218.44" y="93.98"/>
+<pinref part="SJ1" gate="1" pin="2"/>
+<wire x1="-223.52" y1="93.98" x2="-218.44" y2="93.98" width="0.1524" layer="91"/>
 </segment>
 </net>
@@
 <wire x1="-246.38" y1="-30.48" x2="-238.76" y2="-30.48" width="0.1524" layer="91"/>
 <wire x1="-238.76" y1="-30.48" x2="-231.14" y2="-30.48" width="0.1524" layer="91"/>
-<pinref part="SBUS" gate="G$2" pin="VCC"/>
+<pinref part="XBUS" gate="G$2" pin="VCC"/>
 <wire x1="-238.76" y1="-30.48" x2="-238.76" y2="-33.02" width="0.1524" layer="91"/>
 <wire x1="-231.14" y1="-30.48" x2="-231.14" y2="-20.32" width="0.1524" layer="91"/>
@@
 <pinref part="P+7" gate="VCC" pin="VCC"/>
 </segment>
+<segment>
+<pinref part="JP2" gate="A" pin="3"/>
+<wire x1="-198.12" y1="91.44" x2="-185.42" y2="91.44" width="0.1524" layer="91"/>
+<wire x1="-185.42" y1="91.44" x2="-185.42" y2="93.98" width="0.1524" layer="91"/>
+<pinref part="P+6" gate="VCC" pin="VCC"/>
+</segment>
 </net>
 <net name="N$2" class="0">
@@
 <wire x1="-101.6" y1="2.54" x2="-73.66" y2="2.54" width="0.1524" layer="91"/>
 <wire x1="-73.66" y1="2.54" x2="-73.66" y2="-20.32" width="0.1524" layer="91"/>
-<pinref part="SBUS" gate="G$1" pin="RO"/>
+<pinref part="XBUS" gate="G$1" pin="RO"/>
 <wire x1="-73.66" y1="-20.32" x2="-20.32" y2="-20.32" width="0.1524" layer="91"/>
 </segment>
@@
 <wire x1="-248.92" y1="58.42" x2="-251.46" y2="58.42" width="0.1524" layer="91"/>
 <wire x1="-251.46" y1="58.42" x2="-251.46" y2="38.1" width="0.1524" layer="91"/>
-<wire x1="-251.46" y1="38.1" x2="-144.78" y2="38.1" width="0.1524" layer="91"/>
+<wire x1="-251.46" y1="38.1" x2="-208.28" y2="38.1" width="0.1524" layer="91"/>
+<wire x1="-208.28" y1="38.1" x2="-144.78" y2="38.1" width="0.1524" layer="91"/>
 <wire x1="-144.78" y1="38.1" x2="-144.78" y2="17.78" width="0.1524" layer="91"/>
 <pinref part="U$1" gate="G$1" pin="A0"/>
 <wire x1="-144.78" y1="17.78" x2="-134.62" y2="17.78" width="0.1524" layer="91"/>
+<wire x1="-208.28" y1="88.9" x2="-208.28" y2="38.1" width="0.1524" layer="91"/>
+<pinref part="JP2" gate="A" pin="4"/>
+<wire x1="-198.12" y1="88.9" x2="-208.28" y2="88.9" width="0.1524" layer="91"/>
+<junction x="-208.28" y="38.1"/>
 </segment>
 </net>
@@
 <wire x1="-248.92" y1="60.96" x2="-254" y2="60.96" width="0.1524" layer="91"/>
 <wire x1="-254" y1="60.96" x2="-254" y2="35.56" width="0.1524" layer="91"/>
-<wire x1="-254" y1="35.56" x2="-147.32" y2="35.56" width="0.1524" layer="91"/>
+<wire x1="-254" y1="35.56" x2="-205.74" y2="35.56" width="0.1524" layer="91"/>
+<wire x1="-205.74" y1="35.56" x2="-147.32" y2="35.56" width="0.1524" layer="91"/>
 <wire x1="-147.32" y1="35.56" x2="-147.32" y2="15.24" width="0.1524" layer="91"/>
 <pinref part="U$1" gate="G$1" pin="A1"/>
 <wire x1="-147.32" y1="15.24" x2="-134.62" y2="15.24" width="0.1524" layer="91"/>
+<wire x1="-205.74" y1="86.36" x2="-205.74" y2="35.56" width="0.1524" layer="91"/>
+<pinref part="JP2" gate="A" pin="5"/>
+<wire x1="-205.74" y1="86.36" x2="-198.12" y2="86.36" width="0.1524" layer="91"/>
+<junction x="-205.74" y="35.56"/>
 </segment>
 </net>
@@
 <net name="N$4" class="0">
 <segment>
-<pinref part="SBUS" gate="G$1" pin="A"/>
+<pinref part="XBUS" gate="G$1" pin="A"/>
 <wire x1="5.08" y1="-30.48" x2="7.62" y2="-30.48" width="0.1524" layer="91"/>
 <wire x1="7.62" y1="-30.48" x2="17.78" y2="-30.48" width="0.1524" layer="91"/>
@@
 <junction x="17.78" y="-30.48"/>
 <wire x1="17.78" y1="-50.8" x2="20.32" y2="-50.8" width="0.1524" layer="91"/>
-<pinref part="J1" gate="G$1" pin="4"/>
+<pinref part="SBUS" gate="G$1" pin="4"/>
 <wire x1="20.32" y1="-50.8" x2="20.32" y2="-60.96" width="0.1524" layer="91"/>
 </segment>
@@
 <pinref part="R1" gate="G$1" pin="1"/>
 <wire x1="7.62" y1="-43.18" x2="7.62" y2="-45.72" width="0.1524" layer="91"/>
-<pinref part="SBUS" gate="G$1" pin="B"/>
+<pinref part="XBUS" gate="G$1" pin="B"/>
 <wire x1="5.08" y1="-25.4" x2="22.86" y2="-25.4" width="0.1524" layer="91"/>
 <wire x1="22.86" y1="-25.4" x2="22.86" y2="-45.72" width="0.1524" layer="91"/>
@@
 <pinref part="R3" gate="G$1" pin="2"/>
 <wire x1="38.1" y1="-27.94" x2="38.1" y2="-25.4" width="0.1524" layer="91"/>
-<pinref part="J1" gate="G$1" pin="3"/>
+<pinref part="SBUS" gate="G$1" pin="3"/>
 <wire x1="22.86" y1="-45.72" x2="22.86" y2="-60.96" width="0.1524" layer="91"/>
 <junction x="22.86" y="-45.72"/>
@@
 <net name="N$8" class="0">
 <segment>
-<pinref part="J1" gate="G$1" pin="5"/>
+<pinref part="SBUS" gate="G$1" pin="5"/>
 <wire x1="17.78" y1="-60.96" x2="17.78" y2="-58.42" width="0.1524" layer="91"/>
 <wire x1="17.78" y1="-58.42" x2="5.08" y2="-58.42" width="0.1524" layer="91"/>
@@
 </segment>
 </net>
+<net name="N$9" class="0">
+<segment>
+<pinref part="IC9" gate="A" pin="SI"/>
+<wire x1="-248.92" y1="86.36" x2="-254" y2="86.36" width="0.1524" layer="91"/>
+<wire x1="-254" y1="86.36" x2="-254" y2="96.52" width="0.1524" layer="91"/>
+<wire x1="-254" y1="96.52" x2="-233.68" y2="96.52" width="0.1524" layer="91"/>
+<pinref part="SJ1" gate="1" pin="1"/>
+<wire x1="-233.68" y1="93.98" x2="-233.68" y2="96.52" width="0.1524" layer="91"/>
+<junction x="-233.68" y="96.52"/>
+<pinref part="JP2" gate="A" pin="1"/>
+<wire x1="-233.68" y1="96.52" x2="-198.12" y2="96.52" width="0.1524" layer="91"/>
+</segment>
+</net>
